Commit message: adding realsense depth camera to robot

File: ros2_ws/src/PandaRobot/panda_ros2_gazebo/urdf/panda_macro.urdf.xacro (robot description, xacro)
@@ -3,4 +3,9 @@
   <!-- XACRO-MACRO of PANDA ROBOT: -->
   <xacro:macro name="panda" params="prefix EE_no">
+    <xacro:property name="height3" value="1" /> <!-- Link 3 -->
+    <xacro:property name="camera_link" value="0.05" /> <!-- Size of square 'camera' box -->
+    <xacro:property name="axel_offset" value="0.05" /> <!-- Space btw top of beam and the each joint -->
+    <!-- Import Rviz colors -->
+    <xacro:include filename="$(find panda_ros2_gazebo)/urdf/materials.xacro" />
     <!-- Load PANDA ROBOT TRANSMISSION file: -->
     <xacro:include filename="$(find panda_ros2_gazebo)/urdf/panda_transmission.xacro" />
@@ -14,4 +19,9 @@
       EE_no="${EE_no}"
     />
+    <!-- Load PANDA ROBOT CAMERA file: -->
+    <xacro:include filename="$(find panda_ros2_gazebo)/urdf/panda_camera.xacro" />
+    <xacro:panda_camera
+      prefix=""
+    />
     <!-- ***** PANDA ROBOT .urdf SERIAL CHAIN ***** -->
     <!-- panda_link0 -->
@@ -375,4 +385,42 @@
       <child link="end_effector_frame"/>
     </joint>
+    <!-- camera-->
+    <link name="camera_link">
+      <collision>
+        <origin xyz="0 0 0" rpy="0 0 0"/>
+        <geometry>
+          <box size="${camera_link} ${camera_link} ${camera_link}"/>
+        </geometry>
+      </collision>
+      <visual>
+        <origin xyz="0 0 0" rpy="0 0 0"/>
+        <geometry>
+          <box size="${camera_link} ${camera_link} ${camera_link}"/>
+        </geometry>
+        <material name="red"/>
+      </visual>
+      <inertial>
+        <mass value="1e-5" />
+        <origin xyz="0 0 0" rpy="0 0 0"/>
+        <inertia ixx="1e-6" ixy="0" ixz="0" iyy="1e-6" iyz="0" izz="1e-6" />
+      </inertial>
+    </link>
+    <joint name="camera_joint" type="fixed">
+      <!-- <axis xyz="1 1 1" /> -->
+      <origin xyz="-0.065 0 0.05" rpy="0 0 0"/>
+      <parent link="end_effector_frame"/>
+      <child link="camera_link"/>
+    </joint>
+    <!-- generate an optical frame http://www.ros.org/reps/rep-0103.html#suffix-frames
+    so that ros and opencv can operate on the camera frame correctly -->
+    <joint name="camera_optical_joint" type="fixed">
+      <!-- these values have to be these values otherwise the gazebo camera image
+      won't be aligned properly with the frame it is supposedly originating fromrpy="${-pi/2} 0 ${-pi/2}"/> -->
+      <origin xyz="0 0 0" rpy="${-pi/2} 0 ${-pi/2}"/>
+      <parent link="camera_link"/>
+      <child link="camera_link_optical"/>
+    </joint>
+    <link name="camera_link_optical">
+    </link>
   </xacro:macro>
 </robot>

Commit message: added pointcould transformation to world

File: ros2_ws/src/PandaRobot/panda_ros2_gazebo/urdf/panda_macro.urdf.xacro (robot description, xacro)
@@ -66,5 +66,5 @@
     <joint name="camera_optical_joint" type="fixed">
         <origin xyz="0 0 0" rpy="-1.57 0 -1.57"/>
-        <parent link="lens"/>
+        <parent link="camera_link"/>
         <child link="camera_link_optical"/>
     </joint>
