Commit message: separated the camera and robot models

File: ros2_ws/src/PandaRobot/panda_ros2_gazebo/urdf/camera.urdf (robot description, URDF)
Before this commit: robot None, 0 links, 0 joints
Links:
- added link camera_link, mass 1e-5; collision box size=0.1 0.15 0.1; visual box size=0.1 0.15 0.1
- added link camera_link_optical
- added link lens, mass 1e-5; collision box size=0.2 0.025 0.025; visual box size=0.2 0.025 0.025
- added link world
Joints:
- added joint camera_optical_joint: type fixed, parent camera_link, child camera_link_optical, origin xyz=0 0 0 rpy=-1.57 0 -1.57
- added joint lens_to_camera: type fixed, parent camera_link, child lens, origin xyz=0.05 0 0 rpy=0 0 0
- added joint world_to_base: type fixed, parent world, child camera_link

File: ros2_ws/src/PandaRobot/panda_ros2_gazebo/urdf/panda.urdf.xacro (robot description, xacro)
@@ -20,13 +20,14 @@
   <xacro:if value="${cell_layout_1}">
     <joint name="world-base_link-fixed" type="fixed">
+      <org xyz="0.0 0.0 0.0" rpy="0.0 0.0 0.0"/>
       <parent link="world"/>
       <child link="panda_link0"/>
     </joint>
-    <joint name="world-camera_link-fixed" type="fixed">
-      <!-- <origin xyz="0 0 1.5" rpy="0 0.6 3.14"/> -->
-      <origin xyz="0.5 0 0.8" rpy="0 0 0"/>
+    <!-- <joint name="world-camera_link-fixed" type="fixed">
+      <origin xyz="0 0 1.5" rpy="0 0.6 3.14"/>
+      <origin xyz="0.0 0 1.35" rpy="0 0.6 1.57"/>
       <parent link="world"/>
       <child link="camera_link"/>
-    </joint>
+    </joint> -->
   </xacro:if>
 </robot>

File: ros2_ws/src/PandaRobot/panda_ros2_gazebo/urdf/panda_macro.urdf.xacro (robot description, xacro)
@@ -7,5 +7,5 @@
     <xacro:property name="axel_offset" value="0.05" /> <!-- Space btw top of beam and the each joint -->
     <!-- Import Rviz colors -->
-    <xacro:include filename="$(find panda_ros2_gazebo)/urdf/materials.xacro" />
+    <!-- <xacro:include filename="$(find panda_ros2_gazebo)/urdf/materials.xacro" /> -->
     <!-- Load PANDA ROBOT TRANSMISSION file: -->
     <xacro:include filename="$(find panda_ros2_gazebo)/urdf/panda_transmission.xacro" />
@@ -20,7 +20,6 @@
     />
     <!-- ***** PANDA ROBOT .urdf SERIAL CHAIN ***** -->
-    <link name="camera_link">
+    <!-- <link name="camera_link">
         <collision>
-            <!-- <origin xyz="0 0 1.5" rpy="0 0.78 0"/> -->
             <geometry>
                 <box size="0.1 0.15 0.1 "/>
@@ -28,5 +27,4 @@
         </collision>
         <visual>
-            <!-- <origin xyz="0 0 1.5" rpy="0 0.78 0"/> -->
             <geometry>
                 <box size="0.1 0.15 0.1 "/>
@@ -38,8 +36,7 @@
             <inertia ixx="1e-6" ixy="0" ixz="0" iyy="1e-6" iyz="0" izz="1e-6" />
         </inertial>
-    </link>
-    <link name="lens">
+    </link> -->
+    <!-- <link name="lens">
         <collision>
-            <!-- <origin xyz="0 0 1.5" rpy="0 0.78 0"/> -->
             <geometry>
                 <box size="0.2 0.025 0.025"/>
@@ -47,5 +44,4 @@
         </collision>
         <visual>
-            <!-- <origin xyz="0 0 1.5" rpy="0 0.78 0"/> -->
             <geometry>
                 <box size="0.2 0.025 0.025"/>
@@ -57,17 +53,17 @@
             <inertia ixx="1e-6" ixy="0" ixz="0" iyy="1e-6" iyz="0" izz="1e-6"/>
         </inertial>
-    </link>
-    <joint name="lens_to_camera" type="fixed">
+    </link> -->
+    <!-- <joint name="lens_to_camera" type="fixed">
         <origin xyz="0.05 0 0" rpy="0 0 3.14"/>
         <parent link="camera_link"/>
         <child link="lens"/>
-    </joint>
-    <link name="camera_link_optical" />
+    </joint> -->
+    <!-- <link name="camera_link_optical" />
     <joint name="camera_optical_joint" type="fixed">
         <origin xyz="0 0 0" rpy="-1.57 0 -1.57"/>
         <parent link="camera_link"/>
         <child link="camera_link_optical"/>
-    </joint>
-    <gazebo reference="camera_link">
+    </joint> -->
+    <!-- <gazebo reference="camera_link">
         <sensor type="depth" name="realsense">
 	        <always_on>1</always_on>
@@ -79,5 +75,5 @@
 	                <width>640</width>
 	                <height>640</height>
-	                <format>B8G8R8</format>  <!--Changed format since channels were inverted, to go back, change to R8G8B8-->
+	                <format>B8G8R8</format>
 	            </image>
 	            <clip>
@@ -116,5 +112,5 @@
         <mu2>0.2</mu2>
         <material> Gazebo/Red </material>
-    </gazebo>
+    </gazebo> -->
     <!-- panda_link0 -->
     <link name="panda_link0">
