Commit message: added camera above the robot model

File: ros2_ws/src/PandaRobot/panda_ros2_gazebo/urdf/panda.urdf.xacro (robot description, xacro)
@@ -14,4 +14,5 @@
     EE_no="${EE_no}"
   />
+  <!-- <xacro:include filename="$(find panda_ros2_gazebo)/urdf/camera_macro.urdf.xacro"/>	 -->
   <!-- Gazebo world link: -->
   <link name="world"/>
@@ -22,4 +23,9 @@
       <child link="panda_link0"/>
     </joint>
+    <joint name="world-camera_link-fixed" type="fixed">
+      <origin xyz="0 0 1.5" rpy="0 0.6 3.14"/>
+      <parent link="world"/>
+      <child link="camera_link"/>
+    </joint>
   </xacro:if>
 </robot>

File: ros2_ws/src/PandaRobot/panda_ros2_gazebo/urdf/panda_macro.urdf.xacro (robot description, xacro)
@@ -19,10 +19,102 @@
       EE_no="${EE_no}"
     />
-    <!-- Load PANDA ROBOT CAMERA file: -->
-    <xacro:include filename="$(find panda_ros2_gazebo)/urdf/panda_camera.xacro" />
-    <xacro:panda_camera
-      prefix=""
-    />
     <!-- ***** PANDA ROBOT .urdf SERIAL CHAIN ***** -->
+    <link name="camera_link">
+        <collision>
+            <!-- <origin xyz="0 0 1.5" rpy="0 0.78 0"/> -->
+            <geometry>
+                <box size="0.1 0.15 0.1 "/>
+            </geometry>
+        </collision>
+        <visual>
+            <!-- <origin xyz="0 0 1.5" rpy="0 0.78 0"/> -->
+            <geometry>
+                <box size="0.1 0.15 0.1 "/>
+            </geometry>
+        </visual>
+        <inertial>
+            <mass value="1e-5"/>
+            <origin xyz="0 0 0" rpy="0 0 0"/>
+            <inertia ixx="1e-6" ixy="0" ixz="0" iyy="1e-6" iyz="0" izz="1e-6" />
+        </inertial>
+    </link>
+    <link name="lens">
+        <collision>
+            <!-- <origin xyz="0 0 1.5" rpy="0 0.78 0"/> -->
+            <geometry>
+                <box size="0.2 0.025 0.025"/>
+            </geometry>
+        </collision>
+        <visual>
+            <!-- <origin xyz="0 0 1.5" rpy="0 0.78 0"/> -->
+            <geometry>
+                <box size="0.2 0.025 0.025"/>
+            </geometry>
+        </visual>
+        <inertial>
+            <mass value="1e-5"/>
+            <origin xyz="0 0 0" rpy="0 0 0"/>
+            <inertia ixx="1e-6" ixy="0" ixz="0" iyy="1e-6" iyz="0" izz="1e-6"/>
+        </inertial>
+    </link>
+    <joint name="lens_to_camera" type="fixed">
+        <origin xyz="0.05 0 0" rpy="0 0 3.14"/>
+        <parent link="camera_link"/>
+        <child link="lens"/>
+    </joint>
+    <link name="camera_link_optical" />
+    <joint name="camera_optical_joint" type="fixed">
+        <origin xyz="0 0 0" rpy="-1.57 0 -1.57"/>
+        <parent link="lens"/>
+        <child link="camera_link_optical"/>
+    </joint>
+    <gazebo reference="camera_link">
+        <sensor type="depth" name="realsense">
+	        <always_on>1</always_on>
+	        <visualize>true</visualize>
+	        <update_rate>0</update_rate>
+	        <camera>
+	            <horizontal_fov>1.047198</horizontal_fov>
+	            <image>
+	                <width>640</width>
+	                <height>480</height>
+	                <format>B8G8R8</format>  <!--Changed format since channels were inverted, to go back, change to R8G8B8-->
+	            </image>
+	            <clip>
+	                <near>0.01</near>
+	                <far>3</far>
+	            </clip>
+	        </camera>
+	        <plugin name="camera_controller" filename="libgazebo_ros_camera.so">
+	            <baseline>0.2</baseline>
+	            <alwaysOn>true</alwaysOn>
+	            <updateRate>0.0</updateRate>
+	            <cameraName>/realsense</cameraName>
+	            <imageTopicName>/realsense/color/image_raw</imageTopicName>
+	            <cameraInfoTopicName>/realsense/color/camera_info</cameraInfoTopicName>
+	            <depthImageTopicName>/realsense/depth/image_raw</depthImageTopicName>
+	            <depthImageInfoTopicName>/realsense/depth/camera_info</depthImageInfoTopicName>
+	            <pointCloudTopicName>/realsense/depth/points</pointCloudTopicName>
+	            <frameName>camera_link_optical</frameName>
+	            <pointCloudCutoff>0.1</pointCloudCutoff>
+	            <pointCloudCutoffMax>3</pointCloudCutoffMax>
+	            <distortionK1>0</distortionK1>
+	            <distortionK2>0</distortionK2>
+	            <distortionK3>0</distortionK3>
+	            <distortionT1>0</distortionT1>
+	            <distortionT2>0</distortionT2>
+	            <CxPrime>0</CxPrime>
+	            <Cx>0</Cx>
+	            <Cy>0</Cy>
+	            <focalLength>0</focalLength>
+	            <hackBaseline>0</hackBaseline>
+	        </plugin>
+        </sensor>
+    </gazebo>
+    <gazebo reference="lens">
+        <mu1>0.2</mu1>
+        <mu2>0.2</mu2>
+        <material> Gazebo/Red </material>
+    </gazebo>
     <!-- panda_link0 -->
     <link name="panda_link0">
@@ -385,42 +477,4 @@
       <child link="end_effector_frame"/>
     </joint>
-    <!-- camera-->
-    <link name="camera_link">
-      <collision>
-        <origin xyz="0 0 0" rpy="0 0 0"/>
-        <geometry>
-          <box size="${camera_link} ${camera_link} ${camera_link}"/>
-        </geometry>
-      </collision>
-      <visual>
-        <origin xyz="0 0 0" rpy="0 0 0"/>
-        <geometry>
-          <box size="${camera_link} ${camera_link} ${camera_link}"/>
-        </geometry>
-        <material name="red"/>
-      </visual>
-      <inertial>
-        <mass value="1e-5" />
-        <origin xyz="0 0 0" rpy="0 0 0"/>
-        <inertia ixx="1e-6" ixy="0" ixz="0" iyy="1e-6" iyz="0" izz="1e-6" />
-      </inertial>
-    </link>
-    <joint name="camera_joint" type="fixed">
-      <!-- <axis xyz="1 1 1" /> -->
-      <origin xyz="-0.065 0 0.05" rpy="0 0 0"/>
-      <parent link="end_effector_frame"/>
-      <child link="camera_link"/>
-    </joint>
-    <!-- generate an optical frame http://www.ros.org/reps/rep-0103.html#suffix-frames
-    so that ros and opencv can operate on the camera frame correctly -->
-    <joint name="camera_optical_joint" type="fixed">
-      <!-- these values have to be these values otherwise the gazebo camera image
-      won't be aligned properly with the frame it is supposedly originating fromrpy="${-pi/2} 0 ${-pi/2}"/> -->
-      <origin xyz="0 0 0" rpy="${-pi/2} 0 ${-pi/2}"/>
-      <parent link="camera_link"/>
-      <child link="camera_link_optical"/>
-    </joint>
-    <link name="camera_link_optical">
-    </link>
   </xacro:macro>
 </robot>

Commit message: moving the shelf to the front of the robot. added light source

File: ros2_ws/src/PandaRobot/panda_ros2_gazebo/urdf/panda.urdf.xacro (robot description, xacro)
@@ -24,5 +24,6 @@
     </joint>
     <joint name="world-camera_link-fixed" type="fixed">
-      <origin xyz="0 0 1.5" rpy="0 0.6 3.14"/>
+      <!-- <origin xyz="0 0 1.5" rpy="0 0.6 3.14"/> -->
+      <origin xyz="0.5 0 0.8" rpy="0 0 0"/>
       <parent link="world"/>
       <child link="camera_link"/>

Commit message: Working GGCNN pipeline with hardcoded bounding boxes

File: ros2_ws/src/PandaRobot/panda_ros2_gazebo/urdf/panda.urdf.xacro (robot description, xacro)
@@ -24,5 +24,5 @@
     </joint>
     <joint name="world-camera_link-fixed" type="fixed">
-      <origin xyz="0 0 1.5" rpy="0 0.6 3.14"/>
+      <origin xyz="0 0 0.75" rpy="0 0 3.14"/>
       <parent link="world"/>
       <child link="camera_link"/>

Commit message: Added new environment setup

File: ros2_ws/src/PandaRobot/panda_ros2_gazebo/urdf/panda.urdf.xacro (robot description, xacro)
@@ -20,12 +20,14 @@
   <xacro:if value="${cell_layout_1}">
     <joint name="world-base_link-fixed" type="fixed">
+      <org xyz="0.0 0.0 0.0" rpy="0.0 0.0 0.0"/>
       <parent link="world"/>
       <child link="panda_link0"/>
     </joint>
-    <joint name="world-camera_link-fixed" type="fixed">
-      <origin xyz="0 0 0.75" rpy="0 0 3.14"/>
+    <!-- <joint name="world-camera_link-fixed" type="fixed">
+      <origin xyz="0 0 1.5" rpy="0 0.6 3.14"/>
+      <origin xyz="0.0 0 1.35" rpy="0 0.6 1.57"/>
       <parent link="world"/>
       <child link="camera_link"/>
-    </joint>
+    </joint> -->
   </xacro:if>
 </robot>

File: ros2_ws/src/PandaRobot/panda_ros2_gazebo/urdf/panda_macro.urdf.xacro (robot description, xacro)
@@ -7,5 +7,5 @@
     <xacro:property name="axel_offset" value="0.05" /> <!-- Space btw top of beam and the each joint -->
     <!-- Import Rviz colors -->
-    <xacro:include filename="$(find panda_ros2_gazebo)/urdf/materials.xacro" />
+    <!-- <xacro:include filename="$(find panda_ros2_gazebo)/urdf/materials.xacro" /> -->
     <!-- Load PANDA ROBOT TRANSMISSION file: -->
     <xacro:include filename="$(find panda_ros2_gazebo)/urdf/panda_transmission.xacro" />
@@ -20,7 +20,6 @@
     />
     <!-- ***** PANDA ROBOT .urdf SERIAL CHAIN ***** -->
-    <link name="camera_link">
+    <!-- <link name="camera_link">
         <collision>
-            <!-- <origin xyz="0 0 1.5" rpy="0 0.78 0"/> -->
             <geometry>
                 <box size="0.1 0.15 0.1 "/>
@@ -28,5 +27,4 @@
         </collision>
         <visual>
-            <!-- <origin xyz="0 0 1.5" rpy="0 0.78 0"/> -->
             <geometry>
                 <box size="0.1 0.15 0.1 "/>
@@ -38,8 +36,7 @@
             <inertia ixx="1e-6" ixy="0" ixz="0" iyy="1e-6" iyz="0" izz="1e-6" />
         </inertial>
-    </link>
-    <link name="lens">
+    </link> -->
+    <!-- <link name="lens">
         <collision>
-            <!-- <origin xyz="0 0 1.5" rpy="0 0.78 0"/> -->
             <geometry>
                 <box size="0.2 0.025 0.025"/>
@@ -47,5 +44,4 @@
         </collision>
         <visual>
-            <!-- <origin xyz="0 0 1.5" rpy="0 0.78 0"/> -->
             <geometry>
                 <box size="0.2 0.025 0.025"/>
@@ -57,17 +53,17 @@
             <inertia ixx="1e-6" ixy="0" ixz="0" iyy="1e-6" iyz="0" izz="1e-6"/>
         </inertial>
-    </link>
-    <joint name="lens_to_camera" type="fixed">
+    </link> -->
+    <!-- <joint name="lens_to_camera" type="fixed">
         <origin xyz="0.05 0 0" rpy="0 0 3.14"/>
         <parent link="camera_link"/>
         <child link="lens"/>
-    </joint>
-    <link name="camera_link_optical" />
+    </joint> -->
+    <!-- <link name="camera_link_optical" />
     <joint name="camera_optical_joint" type="fixed">
         <origin xyz="0 0 0" rpy="-1.57 0 -1.57"/>
-        <parent link="lens"/>
+        <parent link="camera_link"/>
         <child link="camera_link_optical"/>
-    </joint>
-    <gazebo reference="camera_link">
+    </joint> -->
+    <!-- <gazebo reference="camera_link">
         <sensor type="depth" name="realsense">
 	        <always_on>1</always_on>
@@ -78,6 +74,6 @@
 	            <image>
 	                <width>640</width>
-	                <height>480</height>
-	                <format>B8G8R8</format>  <!--Changed format since channels were inverted, to go back, change to R8G8B8-->
+	                <height>640</height>
+	                <format>B8G8R8</format>
 	            </image>
 	            <clip>
@@ -116,5 +112,5 @@
         <mu2>0.2</mu2>
         <material> Gazebo/Red </material>
-    </gazebo>
+    </gazebo> -->
     <!-- panda_link0 -->
     <link name="panda_link0">
