Commit message: implemented three objects. adjusted camera pose. corrected pcl segmentation

File: ros2_ws/src/PandaRobot/panda_ros2_gazebo/urdf/camera.urdf.xacro (robot description, xacro)
@@ -24,5 +24,6 @@
     <joint name="world_to_base" type="fixed">
       <!-- <origin xyz="0 0 1.5" rpy="0 0.6 3.14"/> -->
-        <origin xyz="0.0 0 1.35" rpy="0 0.6 1.57"/>
+        <!-- <origin xyz="0.0 0 1.35" rpy="0 0.6 1.57"/> -->
+        <origin xyz="-0.3 0 1.0" rpy="0 0.4 1.0"/>
         <parent link="world"/>
         <child link="camera_link"/>

Commit message: corrected sequences to clear objects. adjusted camera position. updated object seg process to remove outliers

File: ros2_ws/src/PandaRobot/panda_ros2_gazebo/urdf/camera.urdf.xacro (robot description, xacro)
@@ -25,5 +25,5 @@
       <!-- <origin xyz="0 0 1.5" rpy="0 0.6 3.14"/> -->
         <!-- <origin xyz="0.0 0 1.35" rpy="0 0.6 1.57"/> -->
-        <origin xyz="-0.3 0 1.0" rpy="0 0.4 1.0"/>
+        <origin xyz="-0.3 0 1.0" rpy="0 0.4 1.2"/>
         <parent link="world"/>
         <child link="camera_link"/>
